File: fixtures/kicad-happy/qualified/control/qualification.kicad_pcb (KiCad board)
At the start: 2 copper layers, 9 parts, among them J1 USB_B, J2 Power, U1 LM317, U2 Load

Commit message: Qualify derating, thermal and EMC adapters with source-backed boundary evidence
Parts:
- R1: value 720 -> 379
- R2: value 240 -> 121
- U1: value LM317 -> TPS7A4501
Connections:
- U1 pad 2: +5V -> +12V
- U1 pad 3: FB -> GND
