File: fixtures/kicad-happy/qualified/protection/qualification.kicad_sch (KiCad schematic)
At the start: 8 parts, among them J1 USB_B, J2 Power, U1 LM317, U2 Load

Commit message: Qualify derating, thermal and EMC adapters with source-backed boundary evidence
Parts:
- R1: value 720 -> 379
- R2: value 240 -> 121
- U1: value LM317 -> TPS7A4501; symbol Regulator_Linear:LM317 -> Regulator_Linear:TPS7A4501
Connections:
- net +12V: now also U1.2 (IN)
- net +5V: now also U1.4 (OUT); no longer U1.2 (VOUT)
- net FB: now also U1.5 (ADJ); no longer U1.3 (ADJ)
- net GND: now also U1.3 (GND), U1.6 (GND)
