File: fixtures/hardware-interface/interface.kicad_sch (KiCad schematic)
At the start: 7 parts, among them X1 port

Commit message: test: declare same-candidate loaded response oracle and supported passive symbols
Parts:
- removed LOAD: 1Meg, symbol Device:R
- added RLOAD: 1Meg, symbol Device:R
- PROBE: symbol Owned:Probe -> ConnectorOwned:Probe
- X1: symbol Owned:Port -> ConnectorOwned:Port
Connections:
- net GND: now also RLOAD.2
- net OUT: now also RLOAD.1
